File: oaed-hardware/high voltage board/Discharging-Circuit.kicad_sch (KiCad schematic)
At the start: 30 parts, among them Q2 IRG7PH35UD, Q3 IRG7PH35UD, Q4 IRG7PH35UD, Q5 IRG7PH35UD, Q6 IRG7PH35UD, Q7 IRG7PH35UD, Q8 IRG7PH35UD, Q9 IRG7PH35UD, U10 TLP250, U11 R1SE/H2_0515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

Commit message: Connect GND and finish symbol updates
Parts:
- Q2, Q3, Q4, Q5, Q6, Q7, Q8, Q9: footprint (none) -> Package_TO_SOT_THT:TO-247-3_Vertical; symbol Q_NIGBT_GCE -> Transistor_IGBT:IRG4PF50W
- U10, U12, U14, U15, U3, U5, U7, U8: footprint DIP-8 -> Package_DIP:DIP-8_W7.62mm; symbol TLP250 -> Driver_FET:TLP250
Connections:
- net +15V: now also U15.8 (VCC), U8.8 (VCC)
- net +VOUT: now also Q3.3 (E), Q4.2 (C), U5.5 (VEE)
- net -VOUT: now also Q7.3 (E), Q8.2 (C), U12.5 (VEE)
- net COUT: now also Q2.2 (C), Q6.2 (C)
- net GND: now also Q5.3 (E), Q9.3 (E), U15.5 (VEE), U8.5 (VEE)
- net at C1.2, U2.4 (-Vout): now also Q2.3 (E), Q3.2 (C), U3.5 (VEE)
- net at C1.1, U2.5 (+Vout): now also U3.8 (VCC)
- net at C2.1, U4.5 (+Vout): now also U5.8 (VCC)
- net at C5.2, U9.4 (-Vout): now also Q6.3 (E), Q7.2 (C), U10.5 (VEE)
- net at C5.1, U9.5 (+Vout): now also U10.8 (VCC)
- net at C6.1, U11.5 (+Vout): now also U12.8 (VCC)
- net at C3.2, U6.4 (-Vout): now also Q4.3 (E), Q5.2 (C), U7.5 (VEE)
- net at C3.1, U6.5 (+Vout): now also U7.8 (VCC)
- net at C7.2, U13.4 (-Vout): now also Q8.3 (E), Q9.2 (C), U14.5 (VEE)
- net at C7.1, U13.5 (+Vout): now also U14.8 (VCC)
- new net: Q2.1 (G), U3.6 (VO), U3.7 (VO)
- new net: Q3.1 (G), U5.6 (VO), U5.7 (VO)
- new net: Q6.1 (G), U10.6 (VO), U10.7 (VO)
- new net: Q7.1 (G), U12.6 (VO), U12.7 (VO)
- new net: Q4.1 (G), U7.6 (VO), U7.7 (VO)
- new net: Q5.1 (G), U8.6 (VO), U8.7 (VO)
- new net: Q8.1 (G), U14.6 (VO), U14.7 (VO)
- new net: Q9.1 (G), U15.6 (VO), U15.7 (VO)
