File: oaed-hardware/high voltage board/High-Voltage-board.kicad_sch (KiCad schematic)
At the start: 1 part

Commit message: Connect GND and finish symbol updates
Changed lines of the file:
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@@
 	)
 	(symbol
-		(lib_id "GND")
+		(lib_id "power:GND")
 		(at 48.26 88.9 0)
 		(unit 1)
@@
 		(on_board yes)
 		(dnp no)
-		(property "Reference" "#PWR1"
+		(fields_autoplaced yes)
+		(property "Reference" "#PWR01"
 			(at 48.26 95.25 0)
 			(effects
@@
 		)
 		(property "Value" "GND"
-			(at 48.26 92.71 0)
+			(at 48.26 93.98 0)
 			(effects
 				(font
@@
 					(size 1.27 1.27)
 				)
+				(hide yes)
 			)
 		)
@@
 					(size 1.27 1.27)
 				)
+				(hide yes)
 			)
 		)
-		(property "Description" ""
+		(property "Description" "Power symbol creates a global label with name \"GND\" , ground"
 			(at 48.26 88.9 0)
 			(effects
@@
 			)
 		)
+		(pin "1"
+		)
 		(instances
 			(project "High-Voltage-board"
 				(path "/04ef437a-7613-4bde-8ffe-10ddaf6e0bfd"
-					(reference "#PWR1")
+					(reference "#PWR01")
 					(unit 1)
 				)
